Commit message: add motors to mjcf

File: description/left_arm_description/urdf/left_arm_description.urdf (robot description, URDF)
Before this commit: robot left_arm_description, 9 links, 8 joints
Joints:
- joint left_joint_4: limit lower=-2.5307 upper=2.5307 effort=12.5 velocity=12.566 -> lower=-2.5307 upper=2.5307 effort=7 velocity=12.566
- joint left_joint_5: limit lower=-0.6981 upper=0.6981 effort=12.5 velocity=12.566 -> lower=-0.6981 upper=0.6981 effort=7 velocity=12.566
- joint left_joint_6: limit lower=-1.5708 upper=1.5708 effort=12.5 velocity=12.566 -> lower=-1.5708 upper=1.5708 effort=7 velocity=12.566
