Commit message: add mojocobridge in python

File: description/dual_arm_support/urdf/dual_arm_robot.urdf (robot description, URDF)
Before this commit: robot dual_arm_robot, 28 links, 27 joints
Joints:
- removed joint leftt_joint_3
- added joint left_joint_3: type revolute, parent left_link_3, child left_link_4, origin xyz=0 0 0 rpy=1.5708 0 0, axis 0 0 1, limit lower=-2.0944 upper=1.4835 effort=27 velocity=3.77

File: description/left_arm_description/urdf/left_arm_description.urdf (robot description, URDF)
Before this commit: robot left_arm_description, 9 links, 8 joints
Joints:
- removed joint leftt_joint_3
- added joint left_joint_3: type revolute, parent left_link_3, child left_link_4, origin xyz=0 0 0 rpy=1.5708 0 0, axis 0 0 1, limit lower=-2.0944 upper=1.4835 effort=27 velocity=3.77

Commit message: add gravity comp controller

File: description/dual_arm_support/urdf/dual_arm_robot.urdf (robot description, URDF)
Before this commit: robot dual_arm_robot, 28 links, 27 joints
Links:
- link left_base_link: mass 0.45399 -> 1.22564
- link left_gripper_gripper_base_link: mass 0.13427 -> 0.35269004
- link left_gripper_left_finger: mass 0.045391 -> 0.04503966
- link left_gripper_right_finger: mass 0.045391 -> 0.04503966
- link left_link_1: mass 0.485026463246757 -> 1.33500720
- link left_link_2: mass 0.0574247036424834 -> 0.18252313
- link left_link_3: mass 0.347887365361116 -> 1.04367671
- link left_link_4: mass 0.192196245053756 -> 0.57070680
- link left_link_5: mass 0.229104472480576 -> 0.66041024
- link left_link_6: mass 0.139362135042712 -> 0.41299778
- link left_link_7: mass 0.0645715321756567 -> 0.19263144
- link right_base_link: mass 0.45399 -> 1.22564018
- link right_gripper_gripper_base_link: mass 0.13427 -> 0.35269004
- link right_gripper_left_finger: mass 0.045391 -> 0.04503966
- link right_gripper_right_finger: mass 0.045391 -> 0.04503966
- link right_link_1: mass 0.48503 -> 1.33502383
- link right_link_2: mass 0.057425 -> 0.18252313
- link right_link_3: mass 0.34789 -> 1.04367487
- link right_link_4: mass 0.1922 -> 0.57070674
- link right_link_5: mass 0.2291 -> 0.66175571
- link right_link_6: mass 0.13936 -> 0.41299783
- link right_link_7: mass 0.064572 -> 0.19263144
Joints:
- joint left_joint_4: limit lower=-2.5307 upper=2.5307 effort=12.5 velocity=12.566 -> lower=-2.5307 upper=2.5307 effort=7.0 velocity=12.566
- joint left_joint_5: limit lower=-0.6981 upper=0.6981 effort=12.5 velocity=12.566 -> lower=-0.6981 upper=0.6981 effort=7.0 velocity=12.566
- joint left_joint_6: limit lower=-1.5708 upper=1.5708 effort=12.5 velocity=12.566 -> lower=-1.5708 upper=1.5708 effort=7.0 velocity=12.566
