Commit message: add right mass info to urdf&mjcf

File: description/gripper_description/urdf/gripper_description.urdf (robot description, URDF)
Before this commit: robot gripper_description, 3 links, 2 joints
Links:
- link gripper_base_link: mass 0.13427 -> 0.35269004
- link left_finger: mass 0.045391 -> 0.04503966
- link right_finger: mass 0.045391 -> 0.04503966

File: description/left_arm_description/urdf/left_arm_description.urdf (robot description, URDF)
Before this commit: robot left_arm_description, 9 links, 8 joints
Links:
- link left_base_link: mass 0.45399 -> 1.22564
- link left_link_1: mass 0.485026463246757 -> 1.33500720
- link left_link_2: mass 0.0574247036424834 -> 0.18252313
- link left_link_3: mass 0.347887365361116 -> 1.04367671
- link left_link_4: mass 0.192196245053756 -> 0.57070680
- link left_link_5: mass 0.229104472480576 -> 0.66041024
- link left_link_6: mass 0.139362135042712 -> 0.41299778
- link left_link_7: mass 0.0645715321756567 -> 0.19263144

File: description/right_arm_description/urdf/right_arm_description.urdf (robot description, URDF)
Before this commit: robot right_arm_description, 9 links, 8 joints
Links:
- link right_base_link: mass 0.45399 -> 1.22564018
- link right_link_1: mass 0.48503 -> 1.33502383
- link right_link_2: mass 0.057425 -> 0.18252313
- link right_link_3: mass 0.34789 -> 1.04367487
- link right_link_4: mass 0.1922 -> 0.57070674
- link right_link_5: mass 0.2291 -> 0.66175571
- link right_link_6: mass 0.13936 -> 0.41299783
- link right_link_7: mass 0.064572 -> 0.19263144
